Commit message: 更新最新版机器人包进度

File: robot description making/MyAttempt_arx_lift2s_description/arx_lift2s_description/urdf/arx_lift2s_ver2.urdf (robot description, URDF)
Before this commit: robot arx_lift2s, 34 links, 33 joints
Links:
- removed link lift_link
- link body_link: mass 1.0 -> 14.181
- link wheel_1: geometry collision mesh filename=package://arx_lift2s_description/meshes/wheel.glb; visual mesh filename=package://arx_lift2s_description/meshes/wheel.glb
- link wheel_2: geometry collision mesh filename=package://arx_lift2s_description/meshes/wheel.glb; visual mesh filename=package://arx_lift2s_description/meshes/wheel.glb
- link wheel_3: geometry collision mesh filename=package://arx_lift2s_description/meshes/wheel.glb; visual mesh filename=package://arx_lift2s_description/meshes/wheel.glb
Joints:
- removed joint lift_joint
- joint arm_left_fixed: origin xyz=0.113964 0.253848 0.012392 rpy=0 0 0 -> xyz=0.059949 0.25 -0.036 rpy=0 0 0; parent lift_link -> body_link
- joint arm_right_fixed: origin xyz=0.113964 -0.246152 0.012392 rpy=0 0 0 -> xyz=0.059949 -0.25 -0.036 rpy=0 0 0; parent lift_link -> body_link
- joint body_joint: limit (none) -> lower=0 upper=0.46 effort=400 velocity=0.15; origin xyz=0.138047 0.001801 0.114163 rpy=0 0 0 -> xyz=0.094118 0.0010067 0.27; parent lift_link -> base_link; type fixed -> prismatic
- joint wheel1_joint: type continuous -> fixed
- joint wheel2_joint: type continuous -> fixed
- joint wheel3_joint: type continuous -> fixed

File: robot description making/MyAttempt_arx_lift2s_description/arx_lift2s_description/urdf/arx_lift2s_ver3.urdf (robot description, URDF)
Before this commit: robot arx_lift2s, 34 links, 33 joints
Links:
- link body_link: mass 1.0 -> 14.181
- link wheel_1: geometry collision mesh filename=package://arx_lift2s_description/meshes/wheel.glb; visual mesh filename=package://arx_lift2s_description/meshes/wheel.glb
- link wheel_2: geometry collision mesh filename=package://arx_lift2s_description/meshes/wheel.glb; visual mesh filename=package://arx_lift2s_description/meshes/wheel.glb
- link wheel_3: geometry collision mesh filename=package://arx_lift2s_description/meshes/wheel.glb; visual mesh filename=package://arx_lift2s_description/meshes/wheel.glb
Joints:
- joint arm_left_fixed: origin xyz=0.113964 0.253848 0.012392 rpy=0 0 0 -> xyz=0.059949 0.25 -0.036 rpy=0 0 0; parent lift_link -> body_link
- joint arm_right_fixed: origin xyz=0.113964 -0.246152 0.012392 rpy=0 0 0 -> xyz=0.059949 -0.25 -0.036 rpy=0 0 0; parent lift_link -> body_link
- joint body_joint: axis 0 0 1 -> (none); origin xyz=0.138047 0.001801 0.114163 rpy=0 0 0 -> xyz=0 0 0 rpy=0 0 0
- joint lift_joint: origin xyz=0.040103 0.0007607 0.221608 -> xyz=0.094118 0.0010067 0.27
- joint wheel1_joint: type continuous -> fixed
- joint wheel2_joint: type continuous -> fixed
- joint wheel3_joint: type continuous -> fixed

File: robot description making/MyAttempt_arx_lift2s_description/arx_lift2s_description/urdf/arx_lift2s_ver4.urdf (robot description, URDF)
Before this commit: robot arx_lift2s, 34 links, 33 joints
Joints:
- joint arm_left_fixed: origin xyz=0.113964 0.253848 0.012392 rpy=0 0 0 -> xyz=0.059949 0.25 -0.036 rpy=0 0 0; parent lift_link -> body_link
- joint arm_right_fixed: origin xyz=0.113964 -0.246152 0.012392 rpy=0 0 0 -> xyz=0.059949 -0.25 -0.036 rpy=0 0 0; parent lift_link -> body_link
- joint body_joint: limit (none) -> lower=0 upper=0 effort=100 velocity=0.1; origin xyz=0.138047 0.001801 0.114163 rpy=0 0 0 -> xyz=0 0 0 rpy=0 0 0; type fixed -> prismatic
- joint lift_joint: origin xyz=0.040103 0.0007607 0.221608 -> xyz=0.094118 0.0010067 0.27
- joint wheel1_joint: type continuous -> fixed
- joint wheel2_joint: type continuous -> fixed
- joint wheel3_joint: type continuous -> fixed

File: robot description making/MyAttempt_arx_lift2s_description/arx_lift2s_description/xacro/components/base.xacro (robot description, xacro)
@@ -1,28 +1,18 @@
 <?xml version="1.0" encoding="utf-8"?>
-<robot xmlns:xacro="http://www.ros.org/wiki/xacro">
-    <!-- 包含轮子模块 -->
+<robot xmlns:xacro="http://www.ros.org/wiki/xacro" name="arx_lift2s_base">
+    <xacro:arg name="robot_name" default="arx_lift2s_base"/>
     <xacro:include filename="$(find arx_lift2s_description)/xacro/components/wheel.xacro"/>
-    <xacro:macro name="Base"  params="enable_wheel_joints:='true'">
+    <xacro:macro name="Base" params="enable_wheel_joints:='true'">
         <link name="base_link">
             <inertial>
                 <origin xyz="-0.010039 0.0013761 0.04956"/>
                 <mass value="21.045"/>
-                <inertia
-                        ixx="1.70029164"
-                        ixy="-0.00073232"
-                        ixz="-0.03255532"
-                        iyy="1.70804910"
-                        iyz="-0.00688370"
-                        izz="0.97173287"/>
+                <inertia ixx="1.70029164" ixy="-0.00073232" ixz="-0.03255532" iyy="1.70804910" iyz="-0.00688370" izz="0.97173287"/>
             </inertial>
             <visual>
-                <geometry>
-                    <mesh filename="file://$(find arx_lift2s_description)/meshes/base_link.glb"/>
-                </geometry>
+                <geometry><mesh filename="file://$(find arx_lift2s_description)/meshes/base_link.glb"/></geometry>
             </visual>
             <collision>
-                <geometry>
-                    <mesh filename="file://$(find arx_lift2s_description)/meshes/base_link.glb"/>
-                </geometry>
+                <geometry><mesh filename="file://$(find arx_lift2s_description)/meshes/base_link.glb"/></geometry>
             </collision>
         </link>
@@ -31,25 +21,15 @@
                 <origin xyz="-0.053315 -0.00061422 -0.0086454"/>
                 <mass value="14.181"/>
-                <inertia
-                        ixx="0.32744849"
-                        ixy="-0.00306617"
-                        ixz="0.05920163"
-                        iyy="0.36541112"
-                        iyz="0.00117932"
-                        izz="0.49616592"/>
+                <inertia ixx="0.32744849" ixy="-0.00306617" ixz="0.05920163" iyy="0.36541112" iyz="0.00117932" izz="0.49616592"/>
             </inertial>
             <visual>
-                <geometry>
-                    <mesh filename="file://$(find arx_lift2s_description)/meshes/body4.glb"/>
-                </geometry>
+                <geometry><mesh filename="file://$(find arx_lift2s_description)/meshes/body4_1.glb"/></geometry>
             </visual>
             <collision>
-                <geometry>
-                    <mesh filename="file://$(find arx_lift2s_description)/meshes/body4.glb"/>
-                </geometry>
+                <geometry><mesh filename="file://$(find arx_lift2s_description)/meshes/body4_1.glb"/></geometry>
             </collision>
         </link>
         <joint name="lift_joint" type="prismatic">
-            <origin xyz="0.094118 0.0010067 0.27"/>
+            <origin xyz="0.040103 0.0007607 0.221608"/>
             <parent link="base_link"/>
             <child link="lift_link"/>
@@ -57,29 +37,40 @@
             <limit lower="0" upper="0.46" effort="400" velocity="0.15"/>
         </joint>
-        <!-- 根据enable_wheel_joints参数决定使用轮子宏还是空link -->
+        <link name="body_link">
+            <inertial>
+                <origin xyz="0 0 0"/>
+                <mass value="1.0"/>
+                <inertia ixx="0.01" ixy="0" ixz="0" iyy="0.01" iyz="0" izz="0.01"/>
+            </inertial>
+            <visual>
+                <geometry><mesh filename="file://$(find arx_lift2s_description)/meshes/body4_2.glb"/></geometry>
+            </visual>
+            <collision>
+                <geometry><mesh filename="file://$(find arx_lift2s_description)/meshes/body4_2.glb"/></geometry>
+            </collision>
+        </link>
+        <joint name="body_joint" type="fixed">
+            <origin xyz="0.138047 0.001801 0.114163" rpy="0 0 0"/>
+            <parent link="lift_link"/>
+            <child link="body_link"/>
+            <axis xyz="0 0 1"/>
+        </joint>
         <xacro:if value="${enable_wheel_joints}">
-            <!-- 启用轮子关节时：使用空link -->
-            <link name="wheel_1"/>
-            <link name="wheel_2"/>
-            <link name="wheel_3"/>
+            <link name="wheel_1"/><link name="wheel_2"/><link name="wheel_3"/>
         </xacro:if>
         <xacro:unless value="${enable_wheel_joints}">
-            <!-- 不启用轮子关节时：使用轮子宏创建完整的轮子link（不包含被动轮） -->
-            <xacro:wheel wheel_name="wheel_1" enable_passive_wheels="false"/>
-            <xacro:wheel wheel_name="wheel_2" enable_passive_wheels="false"/>
-            <xacro:wheel wheel_name="wheel_3" enable_passive_wheels="false"/>
+            <xacro:wheel wheel_name="wheel_1" enable_passive_wheels="false" mesh_rpy="0 0 0"/>
+            <xacro:wheel wheel_name="wheel_2" enable_passive_wheels="false" mesh_rpy="0 0 0"/>
+            <xacro:wheel wheel_name="wheel_3" enable_passive_wheels="false" mesh_rpy="0 0 ${pi}"/>
         </xacro:unless>
-        <xacro:property name="wheel_joint_type" value="fixed"/>
+        <xacro:property name="wheel_joint_type" value="continuous"/>
         <xacro:if value="${enable_wheel_joints}">
             <xacro:property name="wheel_joint_type" value="continuous"/>
         </xacro:if>
-        <!-- 轮子关节定义 -->
         <joint name="wheel1_joint" type="${wheel_joint_type}">
             <origin xyz="0.15361 0.29246 -0.093" rpy="0.0 0.0 1.0472"/>
             <parent link="base_link"/>
             <child link="wheel_1"/>
-            <xacro:if value="${enable_wheel_joints}">
-                <axis xyz="1 0 0"/>
-            </xacro:if>
+            <xacro:if value="${enable_wheel_joints}"><axis xyz="1 0 0"/></xacro:if>
         </joint>
         <joint name="wheel2_joint" type="${wheel_joint_type}">
@@ -87,7 +78,5 @@
             <parent link="base_link"/>
             <child link="wheel_2"/>
-            <xacro:if value="${enable_wheel_joints}">
-                <axis xyz="1 0 0"/>
-            </xacro:if>
+            <xacro:if value="${enable_wheel_joints}"><axis xyz="1 0 0"/></xacro:if>
         </joint>
         <joint name="wheel3_joint" type="${wheel_joint_type}">
@@ -95,7 +84,5 @@
             <parent link="base_link"/>
             <child link="wheel_3"/>
-            <xacro:if value="${enable_wheel_joints}">
-                <axis xyz="-1 0 0"/>
-            </xacro:if>
+            <xacro:if value="${enable_wheel_joints}"><axis xyz="-1 0 0"/></xacro:if>
         </joint>
     </xacro:macro>

File: robot description making/MyAttempt_arx_lift2s_description/arx_lift2s_description/xacro/components/wheel.xacro (robot description, xacro)
@@ -1,13 +1,10 @@
-<?xml version="1.0" encoding="utf-8"?>
+<?xml version="1.0"?>
 <robot xmlns:xacro="http://www.ros.org/wiki/xacro">
     <xacro:property name="PI" value="3.1415926535897931"/>
-    <!-- 被动轮宏定义 -->
     <xacro:macro name="passive_wheel" params="parent_link passive_wheel_name radius angle sphere_radius:='0.06'">
-        <!-- 被动轮链接 -->
         <link name="${passive_wheel_name}">
             <inertial>
                 <origin xyz="0 0 0"/>
-                <mass value="0.1"/>
-                <inertia ixx="0.0001" ixy="0.0" ixz="0.0" iyy="0.0001" iyz="0.0" izz="0.0001"/>
+                <mass value="0.01"/> <inertia ixx="0.0001" ixy="0.0" ixz="0.0" iyy="0.0001" iyz="0.0" izz="0.0001"/>
             </inertial>
             <collision>
@@ -17,7 +14,5 @@
             </collision>
         </link>
-        <!-- 被动轮关节 - 绕x轴旋转，在yz平面上分布，y轴负方向指向圆心 -->
-        <joint name="${passive_wheel_name}_joint" type="continuous">
-            <!-- 让y轴负方向指向圆心：被动轮在角度angle位置，需要绕x轴旋转angle角度使y轴负方向指向圆心 -->
+        <joint name="${passive_wheel_name}_joint" type="fixed">
             <origin xyz="0 ${float(radius) * cos(float(angle))} ${float(radius) * sin(float(angle))}" rpy="${float(angle)} 0 0"/>
             <parent link="${parent_link}"/>
@@ -26,12 +21,8 @@
         </joint>
     </xacro:macro>
-    <!-- 递归宏：创建被动轮循环 -->
     <xacro:macro name="create_passive_wheels" params="parent_link wheel_name indices:=^ angle_step passive_wheel_radius_actual">
         <xacro:if value="${indices}">
-            <!-- 弹出第一个索引 -->
             <xacro:property name="index" value="${indices.pop(0)}"/>
-            <!-- 计算角度 -->
             <xacro:property name="angle" value="${float(index) * float(angle_step)}"/>
-            <!-- 创建被动轮 -->
             <xacro:passive_wheel
                     parent_link="${parent_link}"
@@ -39,5 +30,4 @@
                     radius="${passive_wheel_radius_actual}"
                     angle="${angle}"/>
-            <!-- 递归调用自己 -->
             <xacro:create_passive_wheels
                     parent_link="${parent_link}"
@@ -48,41 +38,43 @@
         </xacro:if>
     </xacro:macro>
-    <!-- 轮子宏定义 - 只包含轮子的link -->
     <xacro:macro name="wheel" params="wheel_name
-                inertial_origin_xyz:='0.035966 2.8161E-06 7.9768E-09'
-                ixx:='0.00142306' ixy:='0.00000000' ixz:='0.00000000' iyy:='0.00084449' iyz:='0.00000002' izz:='0.00084474'
-                passive_wheel_radius:='0.02' wheel_radius:='0.15' num_passive_wheels:='10'
-                enable_passive_wheels:='false'">
-        <!-- 轮子链接 -->
+                                    enable_passive_wheels:='false'
+                                    mesh_rpy:='0 0 0'
+                                    passive_wheel_radius:='0.02'
+                                    num_passive_wheels:='10'">
         <link name="${wheel_name}">
             <inertial>
-                <origin xyz="${inertial_origin_xyz}"/>
-                <mass value="0.5746"/>
-                <inertia ixx="${ixx}" ixy="${ixy}" ixz="${ixz}" iyy="${iyy}" iyz="${iyz}" izz="${izz}"/>
+                <origin xyz="0.035966 2.6831E-06 8.693E-07" rpy="${mesh_rpy}" />
+                <mass value="0.5746" />
+                <inertia
+                        ixx="0.00142306"
+                        ixy="0.00000000"
+                        ixz="0.00000000"
+                        iyy="0.00084449"
+                        iyz="0.00000002"
+                        izz="0.00084474" />
             </inertial>
             <visual>
+                <origin xyz="0 0 0" rpy="${mesh_rpy}" />
                 <geometry>
-                    <mesh filename="file://$(find arx_lift2s_description)/meshes/${wheel_name}.glb"/>
+                    <mesh filename="file://$(find arx_lift2s_description)/meshes/wheel.glb" />
                 </geometry>
             </visual>
             <collision>
+                <origin xyz="0 0 0" rpy="${mesh_rpy}" />
                 <geometry>
-                    <mesh filename="file://$(find arx_lift2s_description)/meshes/${wheel_name}.glb"/>
+                    <mesh filename="file://$(find arx_lift2s_description)/meshes/wheel.glb" />
                 </geometry>
             </collision>
         </link>
-        <!-- 根据参数决定是否创建被动轮 -->
         <xacro:if value="${enable_passive_wheels}">
-            <!-- 创建10个绕一圈的被动轮 -->
             <xacro:property name="num_passive_wheels_float" value="${float(num_passive_wheels)}"/>
             <xacro:property name="angle_step" value="${2*PI / num_passive_wheels_float}"/>
-            <xacro:property name="passive_wheel_radius_actual" value="0.02"/>
-            <xacro:property name="indices" value="${[0,1,2,3,4,5,6,7,8,9]}"/>
-            <xacro:create_passive_wheels
-                    parent_link="${wheel_name}"
-                    wheel_name="${wheel_name}"
-                    indices="${list(indices)}"
-                    angle_step="${angle_step}"
-                    passive_wheel_radius_actual="${passive_wheel_radius_actual}"/>
+            <xacro:property name="indices" value="${[0,1,2,3,4,5,6,7,8,9]}"/> <xacro:create_passive_wheels
+                parent_link="${wheel_name}"
+                wheel_name="${wheel_name}"
+                indices="${list(indices)}"
+                angle_step="${angle_step}"
+                passive_wheel_radius_actual="${passive_wheel_radius}"/>
         </xacro:if>
     </xacro:macro>

File: robot description making/MyAttempt_arx_lift2s_description/arx_lift2s_description/xacro/robot.xacro (robot description, xacro)
@@ -2,25 +2,38 @@
     <xacro:arg name="type" default="x5"/>
     <xacro:arg name="enable_wheel_joints" default="false"/>
-    <xacro:include filename="$(find arx_lift2s_description)/xacro/components/base.xacro"/>
-    <xacro:Base enable_wheel_joints="$(arg enable_wheel_joints)"/>
-    <xacro:if value="${'$(arg type)' == 'x5'}">
-        <xacro:include filename="$(find arx5_description)/xacro/X5.xacro"/>
-        <xacro:X5 name="left"/>
-        <xacro:X5 name="right"/>
+    <xacro:arg name="ros2_control_hardware_type" default="mock_components"/>
+    <xacro:unless value="${'$(arg type)' == 'wheel'}">
+        <xacro:include filename="$(find arx_lift2s_description)/xacro/components/base.xacro"/>
+        <xacro:Base enable_wheel_joints="$(arg enable_wheel_joints)"/>
+        <xacro:if value="${'$(arg type)' == 'x5'}">
+            <xacro:include filename="$(find arx5_description)/xacro/X5.xacro"/>
+            <xacro:X5 name="left"/>
+            <xacro:X5 name="right"/>
+        </xacro:if>
+        <xacro:if value="${'$(arg type)' == 'r5'}">
+            <xacro:include filename="$(find arx5_description)/xacro/R5.xacro"/>
+            <xacro:R5 name="left"/>
+            <xacro:R5 name="right"/>
+        </xacro:if>
+        <joint name="arm_left_fixed" type="fixed">
+            <parent link="lift_link"/>
+            <child link="left_base_link"/>
+            <origin xyz="0.113964 0.253848 0.012392" rpy="0 0 0"/>
+        </joint>
+        <joint name="arm_right_fixed" type="fixed">
+            <parent link="lift_link"/>
+            <child link="right_base_link"/>
+            <origin xyz="0.113964 -0.246152 0.012392" rpy="0 0 0"/>
+        </joint>
+    </xacro:unless>
+    <xacro:if value="${'$(arg type)' == 'wheel'}">
+        <xacro:include filename="$(find arx_lift2s_description)/xacro/components/wheel.xacro"/>
+        <link name="world"/>
+        <xacro:wheel wheel_name="wheel_test" enable_passive_wheels="false"/>
+        <joint name="world_to_wheel" type="fixed">
+            <parent link="world"/>
+            <child link="wheel_test"/>
+            <origin xyz="0 0 0" rpy="0 0 0"/>
+        </joint>
     </xacro:if>
-    <xacro:if value="${'$(arg type)' == 'r5'}">
-        <xacro:include filename="$(find arx5_description)/xacro/R5.xacro"/>
-        <xacro:R5 name="left"/>
-        <xacro:R5 name="right"/>
-    </xacro:if>
-    <joint name="arm_left_fixed" type="fixed">
-        <parent link="lift_link"/>
-        <child link="left_base_link"/>
-        <origin xyz="0.059949 0.25 -0.036" rpy="0 0 0"/>
-    </joint>
-    <joint name="arm_right_fixed" type="fixed">
-        <parent link="lift_link"/>
-        <child link="right_base_link"/>
-        <origin xyz="0.059949 -0.25 -0.036" rpy="0 0 0"/>
-    </joint>
 </robot>
