Commit message: 机器人包所有指令均已跑通

File: robot description making/MyAttempt_arx_lift2s_description/arx_lift2s_description/urdf/arx_lift2s.urdf (robot description, URDF)
Before this commit: robot arx_lift2s, 34 links, 33 joints
Joints:
- joint wheel1_joint: axis (none) -> 1 0 0
- joint wheel2_joint: axis (none) -> 1 0 0
- joint wheel3_joint: axis (none) -> -1 0 0

File: robot description making/MyAttempt_arx_lift2s_description/arx_lift2s_description/xacro/components/base.xacro (robot description, xacro)
@@ -3,5 +3,5 @@
     <xacro:arg name="robot_name" default="arx_lift2s_base"/>
     <xacro:include filename="$(find arx_lift2s_description)/xacro/components/wheel.xacro"/>
-    <xacro:macro name="Base" params="enable_wheel_joints:='true'">
+    <xacro:macro name="Base" params="enable_wheel_joints:='false'">
         <link name="base_link">
             <inertial>
@@ -57,33 +57,26 @@
         </joint>
         <xacro:if value="${enable_wheel_joints}">
-            <link name="wheel_1"/><link name="wheel_2"/><link name="wheel_3"/>
-        </xacro:if>
-        <xacro:unless value="${enable_wheel_joints}">
             <xacro:wheel wheel_name="wheel_1" enable_passive_wheels="false" mesh_rpy="0 0 0"/>
             <xacro:wheel wheel_name="wheel_2" enable_passive_wheels="false" mesh_rpy="0 0 0"/>
             <xacro:wheel wheel_name="wheel_3" enable_passive_wheels="false" mesh_rpy="0 0 ${pi}"/>
-        </xacro:unless>
-        <xacro:property name="wheel_joint_type" value="continuous"/>
-        <xacro:if value="${enable_wheel_joints}">
-            <xacro:property name="wheel_joint_type" value="continuous"/>
+            <joint name="wheel1_joint" type="fixed">
+                <origin xyz="0.15361 0.29246 -0.093" rpy="0.0 0.0 1.0472"/>
+                <parent link="base_link"/>
+                <child link="wheel_1"/>
+                <axis xyz="1 0 0"/>
+            </joint>
+            <joint name="wheel2_joint" type="fixed">
+                <origin xyz="0.15361 -0.29245 -0.093" rpy="0.0 0.0 -1.0472"/>
+                <parent link="base_link"/>
+                <child link="wheel_2"/>
+                <axis xyz="1 0 0"/>
+            </joint>
+            <joint name="wheel3_joint" type="fixed">
+                <origin xyz="-0.35293 0 -0.093" rpy="0.0 0.0 0"/>
+                <parent link="base_link"/>
+                <child link="wheel_3"/>
+                <axis xyz="-1 0 0"/>
+            </joint>
         </xacro:if>
-        <joint name="wheel1_joint" type="${wheel_joint_type}">
-            <origin xyz="0.15361 0.29246 -0.093" rpy="0.0 0.0 1.0472"/>
-            <parent link="base_link"/>
-            <child link="wheel_1"/>
-            <xacro:if value="${enable_wheel_joints}"><axis xyz="1 0 0"/></xacro:if>
-        </joint>
-        <joint name="wheel2_joint" type="${wheel_joint_type}">
-            <origin xyz="0.15361 -0.29245 -0.093" rpy="0.0 0.0 -1.0472"/>
-            <parent link="base_link"/>
-            <child link="wheel_2"/>
-            <xacro:if value="${enable_wheel_joints}"><axis xyz="1 0 0"/></xacro:if>
-        </joint>
-        <joint name="wheel3_joint" type="${wheel_joint_type}">
-            <origin xyz="-0.35293 0 -0.093" rpy="0.0 0.0 0"/>
-            <parent link="base_link"/>
-            <child link="wheel_3"/>
-            <xacro:if value="${enable_wheel_joints}"><axis xyz="-1 0 0"/></xacro:if>
-        </joint>
     </xacro:macro>
 </robot>

File: robot description making/MyAttempt_arx_lift2s_description/arx_lift2s_description/xacro/components/wheel.xacro (robot description, xacro)
@@ -14,5 +14,5 @@
             </collision>
         </link>
-        <joint name="${passive_wheel_name}_joint" type="fixed">
+        <joint name="${passive_wheel_name}_joint" type="continuous">
             <origin xyz="0 ${float(radius) * cos(float(angle))} ${float(radius) * sin(float(angle))}" rpy="${float(angle)} 0 0"/>
             <parent link="${parent_link}"/>

File: robot description making/MyAttempt_arx_lift2s_description/arx_lift2s_description/xacro/robot.xacro (robot description, xacro)
@@ -1,5 +1,5 @@
 <robot name="arx_lift2s" xmlns:xacro="http://www.ros.org/wiki/xacro">
     <xacro:arg name="type" default="x5"/>
-    <xacro:arg name="enable_wheel_joints" default="false"/>
+    <xacro:arg name="enable_wheel_joints" default="true"/>
     <xacro:arg name="ros2_control_hardware_type" default="mock_components"/>
     <xacro:unless value="${'$(arg type)' == 'wheel'}">

File: robot description making/MyAttempt_arx_lift2s_description/arx_lift2s_description/xacro/ros2_control/interfaces.xacro (robot description, xacro)
@@ -10,23 +10,4 @@
             <state_interface name="effort"/>
         </joint>
-        <!-- 移动关节接口定义（注意：lift2s有3个轮子关节） -->
-        <joint name="wheel1_joint">
-            <command_interface name="velocity"/>
-            <state_interface name="position"/>
-            <state_interface name="velocity"/>
-            <state_interface name="effort"/>
-        </joint>
-        <joint name="wheel2_joint">
-            <command_interface name="velocity"/>
-            <state_interface name="position"/>
-            <state_interface name="velocity"/>
-            <state_interface name="effort"/>
-        </joint>
-        <joint name="wheel3_joint">
-            <command_interface name="velocity"/>
-            <state_interface name="position"/>
-            <state_interface name="velocity"/>
-            <state_interface name="effort"/>
-        </joint>
     </xacro:macro>
 </robot>

File: robot description making/MyAttempt_arx_lift2s_description/arx_lift2s_description/xacro/ros2_control/robot.xacro (robot description, xacro)
@@ -4,5 +4,4 @@
     <xacro:arg name="enable_wheel_joints" default="false"/>
     <xacro:arg name="ros2_control_hardware_type" default="mock_components"/>
-    <xacro:arg name="gazebo" default="false" />
     <xacro:include filename="$(find arx_lift2s_description)/xacro/robot.xacro"/>
     <xacro:include filename="$(find arx5_description)/xacro/ros2_control/interfaces.xacro"/>
